Commit message: Fix duplicate aluminum material in mobile_robot URDF
_l515.urdf.xacro already includes _materials.urdf.xacro, so re-including
it at the top level produced two <material name="aluminum"> tags. xacro
does not deduplicate includes, and the URDF parser used by
robot_state_publisher rejects the result with "material 'aluminum' is
not unique", which prevents /robot_description from being published and
blocks Gazebo spawn.

Co-Authored-By: Claude Opus 4.7 (1M context) <noreply@anthropic.com>

File: realsense2_description/urdf/example_mobile_robot_with_l515.urdf.xacro (robot description, xacro)
@@ -12,8 +12,9 @@
 -->
 <robot name="mobile_robot_with_l515" xmlns:xacro="http://ros.org/wiki/xacro">
-  <!-- Include the L515 sensor macro -->
+  <!-- Include the L515 sensor macro. _l515.urdf.xacro already pulls in
+       _materials.urdf.xacro, so we must not include materials a second
+       time here — xacro has no include guard and a duplicate <material>
+       tag fails URDF parsing in robot_state_publisher. -->
   <xacro:include filename="$(find realsense2_description)/urdf/_l515.urdf.xacro" />
-  <!-- Include materials for visualization -->
-  <xacro:include filename="$(find realsense2_description)/urdf/_materials.urdf.xacro" />
   <!-- Constants for robot dimensions -->
   <xacro:property name="base_length" value="0.6" />
